File: project/Power_supply/LLC/lllc.brd (EAGLE design)
At the start: 100 x 80 mm, 2 parts

Commit message: default grid setting
Parts:
- added R1, R2: 50, CasaLibrary:R0805
- added R3, R4: 10k, CasaLibrary:R0805
- added U$3: IRFR024ND2, CasaLibrary:D2PACK
- U$1: value IRFR024N -> TPS92020; device CasaLibrary:D-PAK_TO252AA -> CasaLibrary:SO08
- U$2: value IRFR024N -> IRFR024ND2; device CasaLibrary:D-PAK_TO252AA -> CasaLibrary:D2PACK
- moved U$2 64.8 mm to (39.4, 47.0)
- moved U$1 22.6 mm to (-33.0, 24.1)
Connections:
- new net N$2: R1.2, R3.2, U$2.1
- new net N$3: R2.2, R4.2, U$3.1
- new net N$4: R4.1, U$3.3
- net N$1: now also R3.1, U$2.3, U$3.2; no longer U$1.3, U$2.2
Changed lines of the file:
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@@
 </autorouter>
 <elements>
-<element name="U$1" library="CasaLibrary" package="D-PAK_TO252AA" value="IRFR024N" x="-19.05" y="6.35"/>
-<element name="U$2" library="CasaLibrary" package="D-PAK_TO252AA" value="IRFR024N" x="-19.05" y="19.05"/>
+<element name="R1" library="CasaLibrary" package="R0805" value="50" x="24.13" y="33.02" rot="R270"/>
+<element name="R2" library="CasaLibrary" package="R0805" value="50" x="39.37" y="30.48"/>
+<element name="R3" library="CasaLibrary" package="R0805" value="10k" x="39.37" y="38.1" rot="R180"/>
+<element name="R4" library="CasaLibrary" package="R0805" value="10k" x="26.67" y="38.1" rot="R180"/>
+<element name="U$1" library="CasaLibrary" package="SO08" value="TPS92020" x="-33.02" y="24.13"/>
+<element name="U$2" library="CasaLibrary" package="D2PACK" value="IRFR024ND2" x="39.37" y="46.99"/>
+<element name="U$3" library="CasaLibrary" package="D2PACK" value="IRFR024ND2" x="26.67" y="46.99"/>
 </elements>
 <signals>
 <signal name="N$1">
-<contactref element="U$1" pad="3"/>
-<contactref element="U$2" pad="2"/>
-<wire x1="-19.05" y1="21.55" x2="-16.77" y2="1.55" width="0" layer="19" extent="1-1"/>
+<contactref element="U$2" pad="3"/>
+<contactref element="U$3" pad="2"/>
+<contactref element="R3" pad="1"/>
+<wire x1="40.27" y1="38.1" x2="41.91" y2="38.1" width="0" layer="19" extent="1-1"/>
+<wire x1="26.67" y1="49.53" x2="40.27" y2="38.1" width="0" layer="19" extent="1-1"/>
+</signal>
+<signal name="N$2">
+<contactref element="R1" pad="2"/>
+<contactref element="U$2" pad="1"/>
+<contactref element="R3" pad="2"/>
+<wire x1="36.83" y1="38.1" x2="38.47" y2="38.1" width="0" layer="19" extent="1-1"/>
+<wire x1="24.13" y1="32.12" x2="36.83" y2="38.1" width="0" layer="19" extent="1-1"/>
+</signal>
+<signal name="N$3">
+<contactref element="R2" pad="2"/>
+<contactref element="U$3" pad="1"/>
+<contactref element="R4" pad="2"/>
+<wire x1="25.77" y1="38.1" x2="40.27" y2="30.48" width="0" layer="19" extent="1-1"/>
+<wire x1="24.13" y1="38.1" x2="25.77" y2="38.1" width="0" layer="19" extent="1-1"/>
+</signal>
+<signal name="N$4">
+<contactref element="R4" pad="1"/>
+<contactref element="U$3" pad="3"/>
+<wire x1="27.57" y1="38.1" x2="29.21" y2="38.1" width="0" layer="19" extent="1-1"/>
 </signal>
 </signals>
