File: project/Power_supply/LLC/lllc.sch (EAGLE design)
At the start: 2 parts

Commit message: default grid setting
Parts:
- added R1, R2: 50, CasaLibrary:R0805
- added R3, R4: 10k, CasaLibrary:R0805
- added U$3: IRFR024ND2, CasaLibrary:IRFR024ND2
- U$1: value IRFR024N -> TPS92020; device CasaLibrary:IRFR024N -> CasaLibrary:TPS92020
- U$2: value IRFR024N -> IRFR024ND2; device CasaLibrary:IRFR024N -> CasaLibrary:IRFR024ND2
Connections:
- new net N$2: R1.2, R3.2, U$2.G
- new net N$3: R2.2, R4.2, U$3.G
- new net N$4: R4.1, U$3.S
- net N$1: now also R3.1, U$2.S, U$3.D; no longer U$1.S, U$2.D
Changed lines of the file:
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@@
 <setting verticaltext="up"/>
 </settings>
-<grid distance="0.1" unitdist="inch" unit="inch" style="lines" multiple="1" display="no" altdistance="0.01" altunitdist="inch" altunit="inch"/>
+<grid distance="0.05" unitdist="inch" unit="inch" style="lines" multiple="1" display="yes" altdistance="0.01" altunitdist="inch" altunit="inch"/>
 <layers>
 <layer number="1" name="Top" color="4" fill="1" visible="no" active="no"/>
@@
 </classes>
 <parts>
-<part name="U$1" library="CasaLibrary" deviceset="IRFR024N" device=""/>
-<part name="U$2" library="CasaLibrary" deviceset="IRFR024N" device=""/>
+<part name="U$1" library="CasaLibrary" deviceset="TPS92020" device=""/>
+<part name="U$2" library="CasaLibrary" deviceset="IRFR024N" device="D2"/>
+<part name="U$3" library="CasaLibrary" deviceset="IRFR024N" device="D2"/>
+<part name="R1" library="CasaLibrary" deviceset="R" device="0805" value="50"/>
+<part name="R2" library="CasaLibrary" deviceset="R" device="0805" value="50"/>
+<part name="R3" library="CasaLibrary" deviceset="R" device="0805" value="10k"/>
+<part name="R4" library="CasaLibrary" deviceset="R" device="0805" value="10k"/>
 </parts>
 <sheets>
@@
 </plain>
 <instances>
-<instance part="U$1" gate="G$1" x="55.88" y="53.34"/>
-<instance part="U$2" gate="G$1" x="55.88" y="35.56"/>
+<instance part="U$1" gate="G$1" x="76.2" y="48.26"/>
+<instance part="U$2" gate="G$1" x="200.66" y="45.72"/>
+<instance part="U$3" gate="G$1" x="200.66" y="21.59"/>
+<instance part="R1" gate="G$1" x="186.69" y="43.18"/>
+<instance part="R2" gate="G$1" x="186.69" y="19.05"/>
+<instance part="R3" gate="G$1" x="193.04" y="36.83" rot="R90"/>
+<instance part="R4" gate="G$1" x="193.04" y="12.7" rot="R90"/>
 </instances>
 <busses>
@@
 <net name="N$1" class="0">
 <segment>
-<pinref part="U$1" gate="G$1" pin="S"/>
-<pinref part="U$2" gate="G$1" pin="D"/>
-<wire x1="55.88" y1="40.64" x2="55.88" y2="48.26" width="0.1524" layer="91"/>
+<pinref part="U$2" gate="G$1" pin="S"/>
+<pinref part="U$3" gate="G$1" pin="D"/>
+<wire x1="200.66" y1="26.67" x2="200.66" y2="30.48" width="0.1524" layer="91"/>
+<pinref part="R3" gate="G$1" pin="1"/>
+<wire x1="200.66" y1="30.48" x2="200.66" y2="40.64" width="0.1524" layer="91"/>
+<wire x1="193.04" y1="31.75" x2="193.04" y2="30.48" width="0.1524" layer="91"/>
+<wire x1="193.04" y1="30.48" x2="200.66" y2="30.48" width="0.1524" layer="91"/>
+</segment>
+</net>
+<net name="N$2" class="0">
+<segment>
+<pinref part="R1" gate="G$1" pin="2"/>
+<pinref part="U$2" gate="G$1" pin="G"/>
+<wire x1="191.77" y1="43.18" x2="193.04" y2="43.18" width="0.1524" layer="91"/>
+<pinref part="R3" gate="G$1" pin="2"/>
+<wire x1="194.31" y1="43.18" x2="193.04" y2="43.18" width="0.1524" layer="91"/>
+<wire x1="193.04" y1="41.91" x2="193.04" y2="43.18" width="0.1524" layer="91"/>
+</segment>
+</net>
+<net name="N$3" class="0">
+<segment>
+<pinref part="R2" gate="G$1" pin="2"/>
+<pinref part="U$3" gate="G$1" pin="G"/>
+<wire x1="191.77" y1="19.05" x2="194.31" y2="19.05" width="0.1524" layer="91"/>
+<pinref part="R4" gate="G$1" pin="2"/>
+<wire x1="194.31" y1="19.05" x2="193.04" y2="19.05" width="0.1524" layer="91"/>
+<wire x1="193.04" y1="19.05" x2="193.04" y2="17.78" width="0.1524" layer="91"/>
+</segment>
+</net>
+<net name="N$4" class="0">
+<segment>
+<pinref part="R4" gate="G$1" pin="1"/>
+<wire x1="193.04" y1="7.62" x2="193.04" y2="6.35" width="0.1524" layer="91"/>
+<pinref part="U$3" gate="G$1" pin="S"/>
+<wire x1="193.04" y1="6.35" x2="200.66" y2="6.35" width="0.1524" layer="91"/>
+<wire x1="200.66" y1="6.35" x2="200.66" y2="16.51" width="0.1524" layer="91"/>
 </segment>
 </net>
 </nets>
 </sheet>
+<sheet>
+<plain>
+</plain>
+<instances>
+</instances>
+<busses>
+</busses>
+<nets>
+</nets>
+</sheet>
